File: mcuPower/eagle_files/dev/mcuPower.sch (EAGLE design)
At the start: 8 parts, among them P1 CR2032, P2 CR2032, U1 PQ070XF01SZH

Commit message: additional tweaks to Eagle files. approaching final. focus here on ease of battery placement and space clearance.
Connections:
- net VCC: now also P2.VCC_3; no longer P2.VCC_2
Changed lines of the file:
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@@
 <net name="VCC" class="0">
 <segment>
-<wire x1="53.34" y1="93.98" x2="53.34" y2="91.44" width="0.1524" layer="91"/>
-<wire x1="53.34" y1="91.44" x2="53.34" y2="60.96" width="0.1524" layer="91"/>
+<wire x1="53.34" y1="93.98" x2="53.34" y2="86.36" width="0.1524" layer="91"/>
+<wire x1="53.34" y1="86.36" x2="53.34" y2="60.96" width="0.1524" layer="91"/>
 <wire x1="53.34" y1="60.96" x2="73.66" y2="60.96" width="0.1524" layer="91"/>
 <wire x1="73.66" y1="60.96" x2="73.66" y2="63.5" width="0.1524" layer="91"/>
@@
 <junction x="53.34" y="60.96"/>
 <pinref part="U1" gate="G$1" pin="VIN"/>
-<wire x1="33.02" y1="91.44" x2="53.34" y2="91.44" width="0.1524" layer="91"/>
-<junction x="53.34" y="91.44"/>
-<pinref part="P2" gate="G$1" pin="VCC_2"/>
+<pinref part="P2" gate="G$1" pin="VCC_3"/>
+<wire x1="33.02" y1="86.36" x2="53.34" y2="86.36" width="0.1524" layer="91"/>
+<junction x="53.34" y="86.36"/>
 </segment>
 </net>
