File: PCB/LightStickPower/eagle_files/dev/LightStickPower.brd (EAGLE design)
At the start: 25 x 15 mm, 7 parts

Commit message: Add traces.
Routing:
- net N$5: track 0.00 -> 66.7 mm
- net N$1: track 0.00 -> 27.0 mm
- net N$3: track 0.00 -> 9.17 mm
- net N$7: track 0.00 -> 9.01 mm
- net N$2: track 0.00 -> 8.89 mm
Changed lines of the file:
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@@
 <contactref element="C2" pad="1"/>
 <contactref element="V1" pad="VIN"/>
-<wire x1="16" y1="5" x2="13.8" y2="13.95" width="0" layer="19" extent="16-16"/>
-<wire x1="2.5" y1="4.4" x2="16" y2="5" width="0" layer="19" extent="1-1"/>
-<wire x1="16.7" y1="6.7" x2="2.5" y2="4.4" width="0" layer="19" extent="1-1"/>
+<wire x1="2.5" y1="4.4" x2="5.69" y2="4.4" width="0.4064" layer="1"/>
+<wire x1="5.69" y1="4.4" x2="8" y2="6.71" width="0.4064" layer="1"/>
+<wire x1="8" y1="6.71" x2="16.69" y2="6.71" width="0.4064" layer="1"/>
+<wire x1="16.69" y1="6.71" x2="16.7" y2="6.7" width="0.4064" layer="1"/>
+<wire x1="16" y1="5" x2="16" y2="6" width="0.4064" layer="1"/>
+<wire x1="16" y1="6" x2="16.7" y2="6.7" width="0.4064" layer="1"/>
+<wire x1="13.8" y1="13.95" x2="13.8" y2="12.7" width="0.4064" layer="16"/>
+<wire x1="13.8" y1="12.7" x2="16" y2="10.5" width="0.4064" layer="16"/>
+<wire x1="16" y1="10.5" x2="16" y2="5" width="0.4064" layer="16"/>
 </signal>
 <signal name="N$2">
 <contactref element="USB1" pad="D-"/>
 <contactref element="USB2" pad="DATA-"/>
-<wire x1="13.5" y1="5" x2="13.15" y2="13.75" width="0" layer="19" extent="16-16"/>
+<wire x1="13.5" y1="5" x2="13.5" y2="11.37" width="0.4064" layer="16"/>
+<wire x1="13.5" y1="11.37" x2="13.17" y2="11.7" width="0.4064" layer="16"/>
+<wire x1="13.17" y1="11.7" x2="13.17" y2="13.73" width="0.4064" layer="16"/>
+<wire x1="13.17" y1="13.73" x2="13.15" y2="13.75" width="0.4064" layer="16"/>
 </signal>
 <signal name="N$3">
 <contactref element="USB1" pad="D+"/>
 <contactref element="USB2" pad="DATA+"/>
-<wire x1="11.5" y1="5" x2="12.5" y2="13.75" width="0" layer="19" extent="16-16"/>
+<wire x1="11.5" y1="5" x2="11.5" y2="10.79" width="0.4064" layer="16"/>
+<wire x1="11.5" y1="10.79" x2="12.51" y2="11.8" width="0.4064" layer="16"/>
+<wire x1="12.51" y1="11.8" x2="12.51" y2="13.74" width="0.4064" layer="16"/>
+<wire x1="12.51" y1="13.74" x2="12.5" y2="13.75" width="0.4064" layer="16"/>
 </signal>
 <signal name="N$7">
@@
 <contactref element="C1" pad="1"/>
 <contactref element="V1" pad="VOUT2"/>
-<wire x1="22.5" y1="4.4" x2="23" y2="13" width="0" layer="19" extent="1-1"/>
-<wire x1="22.25" y1="9" x2="22.5" y2="4.4" width="0" layer="19" extent="1-1"/>
+<wire x1="22.5" y1="4.4" x2="22.5" y2="8.75" width="0.4064" layer="1"/>
+<wire x1="22.5" y1="8.75" x2="22.25" y2="9" width="0.4064" layer="1"/>
+<wire x1="22.25" y1="9" x2="22.25" y2="12.25" width="0.4064" layer="1"/>
+<wire x1="22.25" y1="12.25" x2="23" y2="13" width="0.4064" layer="1"/>
 </signal>
 <signal name="N$5">
@@
 <contactref element="USB2" pad="GND"/>
 <contactref element="V1" pad="GND"/>
-<wire x1="9" y1="5" x2="22.5" y2="2.6" width="0" layer="19" extent="1-1"/>
-<wire x1="2.5" y1="2.6" x2="9" y2="5" width="0" layer="19" extent="1-1"/>
-<wire x1="11.2" y1="13.95" x2="9" y2="5" width="0" layer="19" extent="16-16"/>
-<wire x1="16.7" y1="11.3" x2="2.5" y2="2.6" width="0" layer="19" extent="1-1"/>
-<wire x1="2" y1="13" x2="11.2" y2="13.95" width="0" layer="19" extent="16-16"/>
+<wire x1="2" y1="13" x2="10.25" y2="13" width="0.4064" layer="16"/>
+<wire x1="10.25" y1="13" x2="11.2" y2="13.95" width="0.4064" layer="16"/>
+<wire x1="9" y1="5" x2="9" y2="11.75" width="0.4064" layer="16"/>
+<wire x1="9" y1="11.75" x2="10.25" y2="13" width="0.4064" layer="16"/>
+<wire x1="2.5" y1="2.6" x2="1.9" y2="2.6" width="0.4064" layer="1"/>
+<wire x1="1.9" y1="2.6" x2="1" y2="3.5" width="0.4064" layer="1"/>
+<wire x1="1" y1="3.5" x2="1" y2="12" width="0.4064" layer="1"/>
+<wire x1="1" y1="12" x2="2" y2="13" width="0.4064" layer="1"/>
+<wire x1="16.7" y1="11.3" x2="3.7" y2="11.3" width="0.4064" layer="1"/>
+<wire x1="3.7" y1="11.3" x2="2" y2="13" width="0.4064" layer="1"/>
+<wire x1="22.5" y1="2.6" x2="22.5" y2="2.5" width="0.4064" layer="1"/>
+<wire x1="22.5" y1="2.5" x2="21" y2="1" width="0.4064" layer="1"/>
+<wire x1="21" y1="1" x2="4.1" y2="1" width="0.4064" layer="1"/>
+<wire x1="4.1" y1="1" x2="2.5" y2="2.6" width="0.4064" layer="1"/>
 </signal>
 </signals>

Commit message: Finalize LightStickPower.
Parts:
- moved USB2 3.10 mm to (12.5, 17.6)
Routing:
- net N$2: track 8.89 -> 12.3 mm
- net N$1: track 27.0 -> 30.3 mm
- net N$5: track 66.7 -> 69.8 mm
- net N$3: track 9.17 -> 12.3 mm
Other:
- board size 25 x 15 mm -> 25 x 18 mm
- board text added: "LightStickPower1.0 8/14/16 F. Lee"
Changed lines of the file:
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@@
 <wire x1="0" y1="0" x2="25" y2="0" width="0" layer="20"/>
 <wire x1="25" y1="0" x2="25" y2="15" width="0" layer="20"/>
-<wire x1="25" y1="15" x2="0" y2="15" width="0" layer="20"/>
 <wire x1="0" y1="15" x2="0" y2="0" width="0" layer="20"/>
+<wire x1="0" y1="15" x2="9" y2="15" width="0" layer="20"/>
+<wire x1="25" y1="15" x2="16" y2="15" width="0" layer="20"/>
+<wire x1="16" y1="15" x2="16" y2="18" width="0" layer="20"/>
+<wire x1="16" y1="18" x2="9" y2="18" width="0" layer="20"/>
+<wire x1="9" y1="18" x2="9" y2="15" width="0" layer="20"/>
+<text x="3.5" y="7" size="0.6096" layer="25">LightStickPower1.0
+8/14/16
+F. Lee</text>
 </plain>
 <attributes>
@@
 </class>
 </classes>
-<designrules name="default">
+<designrules name="LaenPCBOrder">
 <description language="de">&lt;b&gt;EAGLE Design Rules&lt;/b&gt;
 &lt;p&gt;
@@
 Einstellungen hier und speichern die Design Rules unter
 einem neuen Namen ab.</description>
-<description language="en">&lt;b&gt;EAGLE Design Rules&lt;/b&gt;
+<description language="en">&lt;b&gt;Laen's PCB Order Design Rules&lt;/b&gt;
 &lt;p&gt;
-The default Design Rules have been set to cover
-a wide range of applications. Your particular design
-may have different requirements, so please make the
-necessary adjustments and save your customized
-design rules under a new name.</description>
+Please make sure your boards conform to these design rules.</description>
 <param name="layerSetup" value="(1*16)"/>
-<param name="mtCopper" value="0.035mm 0.035mm 0.035mm 0.035mm 0.035mm 0.035mm 0.035mm 0.035mm 0.035mm 0.035mm 0.035mm 0.035mm 0.035mm 0.035mm 0.035mm 0.035mm"/>
-<param name="mtIsolate" value="1.5mm 0.15mm 0.2mm 0.15mm 0.2mm 0.15mm 0.2mm 0.15mm 0.2mm 0.15mm 0.2mm 0.15mm 0.2mm 0.15mm 0.2mm"/>
-<param name="mdWireWire" value="8mil"/>
-<param name="mdWirePad" value="8mil"/>
-<param name="mdWireVia" value="8mil"/>
-<param name="mdPadPad" value="8mil"/>
-<param name="mdPadVia" value="8mil"/>
-<param name="mdViaVia" value="8mil"/>
-<param name="mdSmdPad" value="8mil"/>
-<param name="mdSmdVia" value="8mil"/>
-<param name="mdSmdSmd" value="8mil"/>
+<param name="mtCopper" value="0.0356mm 0.0356mm 0.0356mm 0.0356mm 0.0356mm 0.0356mm 0.0356mm 0.0356mm 0.0356mm 0.0356mm 0.0356mm 0.0356mm 0.0356mm 0.0356mm 0.0356mm 0.0356mm"/>
+<param name="mtIsolate" value="1.5011mm 0.1499mm 0.2007mm 0.1499mm 0.2007mm 0.1499mm 0.2007mm 0.1499mm 0.2007mm 0.1499mm 0.2007mm 0.1499mm 0.2007mm 0.1499mm 0.2007mm"/>
+<param name="mdWireWire" value="6mil"/>
+<param name="mdWirePad" value="6mil"/>
+<param name="mdWireVia" value="6mil"/>
+<param name="mdPadPad" value="6mil"/>
+<param name="mdPadVia" value="6mil"/>
+<param name="mdViaVia" value="6mil"/>
+<param name="mdSmdPad" value="6mil"/>
+<param name="mdSmdVia" value="6mil"/>
+<param name="mdSmdSmd" value="6mil"/>
 <param name="mdViaViaSameLayer" value="8mil"/>
 <param name="mnLayersViaInSmd" value="2"/>
-<param name="mdCopperDimension" value="40mil"/>
-<param name="mdDrill" value="8mil"/>
+<param name="mdCopperDimension" value="15mil"/>
+<param name="mdDrill" value="6mil"/>
 <param name="mdSmdStop" value="0mil"/>
-<param name="msWidth" value="10mil"/>
-<param name="msDrill" value="24mil"/>
-<param name="msMicroVia" value="9.99mm"/>
+<param name="msWidth" value="6mil"/>
+<param name="msDrill" value="13mil"/>
+<param name="msMicroVia" value="13mil"/>
 <param name="msBlindViaRatio" value="0.5"/>
 <param name="rvPadTop" value="0.25"/>
@@
 <param name="rvMicroViaOuter" value="0.25"/>
 <param name="rvMicroViaInner" value="0.25"/>
-<param name="rlMinPadTop" value="10mil"/>
+<param name="rlMinPadTop" value="7mil"/>
 <param name="rlMaxPadTop" value="20mil"/>
-<param name="rlMinPadInner" value="10mil"/>
+<param name="rlMinPadInner" value="7mil"/>
 <param name="rlMaxPadInner" value="20mil"/>
-<param name="rlMinPadBottom" value="10mil"/>
+<param name="rlMinPadBottom" value="7mil"/>
 <param name="rlMaxPadBottom" value="20mil"/>
-<param name="rlMinViaOuter" value="8mil"/>
+<param name="rlMinViaOuter" value="7mil"/>
 <param name="rlMaxViaOuter" value="20mil"/>
-<param name="rlMinViaInner" value="8mil"/>
+<param name="rlMinViaInner" value="7mil"/>
 <param name="rlMaxViaInner" value="20mil"/>
 <param name="rlMinMicroViaOuter" value="4mil"/>
@@
 <param name="mvStopFrame" value="1"/>
 <param name="mvCreamFrame" value="0"/>
-<param name="mlMinStopFrame" value="4mil"/>
-<param name="mlMaxStopFrame" value="4mil"/>
+<param name="mlMinStopFrame" value="3mil"/>
+<param name="mlMaxStopFrame" value="3mil"/>
 <param name="mlMinCreamFrame" value="0mil"/>
 <param name="mlMaxCreamFrame" value="0mil"/>
@@
 <attribute name="NAME" x="4.25" y="5" size="1.27" layer="25" rot="R270"/>
 </element>
-<element name="USB2" library="freddyLibr" package="USB_MICROB_PLUG_ZX64_B_5S" value="USB_MICROB_PLUG_ZX64_B_5S" x="12.5" y="14.5" smashed="yes" rot="MR180">
-<attribute name="NAME" x="10.24" y="12.5" size="1.27" layer="26" rot="MR0"/>
+<element name="USB2" library="freddyLibr" package="USB_MICROB_PLUG_ZX64_B_5S" value="USB_MICROB_PLUG_ZX64_B_5S" x="12.5" y="17.6" smashed="yes" rot="MR180">
+<attribute name="NAME" x="14.3" y="13.24" size="1.27" layer="26" rot="MR90"/>
 </element>
 <element name="GND" library="SparkFun-Connectors" package="1X01" value="" x="2" y="13" smashed="yes">
@@
 <wire x1="16" y1="5" x2="16" y2="6" width="0.4064" layer="1"/>
 <wire x1="16" y1="6" x2="16.7" y2="6.7" width="0.4064" layer="1"/>
-<wire x1="13.8" y1="13.95" x2="13.8" y2="12.7" width="0.4064" layer="16"/>
-<wire x1="13.8" y1="12.7" x2="16" y2="10.5" width="0.4064" layer="16"/>
-<wire x1="16" y1="10.5" x2="16" y2="5" width="0.4064" layer="16"/>
+<wire x1="13.8" y1="17.05" x2="13.8" y2="16.19" width="0.4064" layer="16"/>
+<wire x1="13.8" y1="16.19" x2="16.17" y2="13.82" width="0.4064" layer="16"/>
+<wire x1="16.17" y1="13.82" x2="16.17" y2="5.17" width="0.4064" layer="16"/>
+<wire x1="16.17" y1="5.17" x2="16" y2="5" width="0.4064" layer="16"/>
 </signal>
 <signal name="N$2">
 <contactref element="USB1" pad="D-"/>
 <contactref element="USB2" pad="DATA-"/>
-<wire x1="13.5" y1="5" x2="13.5" y2="11.37" width="0.4064" layer="16"/>
-<wire x1="13.5" y1="11.37" x2="13.17" y2="11.7" width="0.4064" layer="16"/>
-<wire x1="13.17" y1="11.7" x2="13.17" y2="13.73" width="0.4064" layer="16"/>
-<wire x1="13.17" y1="13.73" x2="13.15" y2="13.75" width="0.4064" layer="16"/>
+<wire x1="13.5" y1="5" x2="13.5" y2="14.97" width="0.4064" layer="16"/>
+<wire x1="13.5" y1="14.97" x2="13.14" y2="15.33" width="0.4064" layer="16"/>
+<wire x1="13.14" y1="15.33" x2="13.14" y2="16.99" width="0.4064" layer="16"/>
+<wire x1="13.14" y1="16.99" x2="13.15" y2="16.85" width="0.4064" layer="16"/>
 </signal>
 <signal name="N$3">
 <contactref element="USB1" pad="D+"/>
 <contactref element="USB2" pad="DATA+"/>
-<wire x1="11.5" y1="5" x2="11.5" y2="10.79" width="0.4064" layer="16"/>
-<wire x1="11.5" y1="10.79" x2="12.51" y2="11.8" width="0.4064" layer="16"/>
-<wire x1="12.51" y1="11.8" x2="12.51" y2="13.74" width="0.4064" layer="16"/>
-<wire x1="12.51" y1="13.74" x2="12.5" y2="13.75" width="0.4064" layer="16"/>
+<wire x1="12.5" y1="16.85" x2="12.5" y2="6" width="0.4064" layer="16"/>
+<wire x1="12.5" y1="6" x2="11.5" y2="5" width="0.4064" layer="16"/>
 </signal>
 <signal name="N$7">
@@
 <contactref element="V1" pad="GND"/>
 <wire x1="2" y1="13" x2="10.25" y2="13" width="0.4064" layer="16"/>
-<wire x1="10.25" y1="13" x2="11.2" y2="13.95" width="0.4064" layer="16"/>
 <wire x1="9" y1="5" x2="9" y2="11.75" width="0.4064" layer="16"/>
 <wire x1="9" y1="11.75" x2="10.25" y2="13" width="0.4064" layer="16"/>
@@
 <wire x1="21" y1="1" x2="4.1" y2="1" width="0.4064" layer="1"/>
 <wire x1="4.1" y1="1" x2="2.5" y2="2.6" width="0.4064" layer="1"/>
+<wire x1="11.2" y1="17.05" x2="11.2" y2="13.95" width="0.4064" layer="16"/>
+<wire x1="11.2" y1="13.95" x2="10.25" y2="13" width="0.4064" layer="16"/>
 </signal>
 </signals>
 </board>
 </drawing>
+<compatibility>
+<note version="6.3" minversion="6.2.2" severity="warning">
+Since Version 6.2.2 text objects can contain more than one line,
+which will not be processed correctly with this version.
+</note>
+</compatibility>
 </eagle>
