File: PCB/LightStickPower/eagle_files/dev/LightStickPower.sch (EAGLE design)
At the start: 7 parts

Commit message: Updated Light stick power to use cabled USB-micro-B plug. Also commit properly pathed copy_eagle. Getting annoying.
Parts:
- removed USB2: USB_MICROB_PLUG_ZX64_B_5S, freddyLibr:USB_MICROB_PLUG_ZX64_B_5S
- added JP1: (no value), SparkFun-Connectors:M04PTH
Connections:
- net N$1: now also JP1.4; no longer USB2.VCC
- net N$2: now also JP1.3; no longer USB2.DATA-
- net N$3: now also JP1.2; no longer USB2.DATA+
- net N$5: now also JP1.1; no longer USB2.GND
Changed lines of the file:
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@@
 <parts>
 <part name="USB1" library="freddyLibr" deviceset="USB_A_932" device=""/>
-<part name="USB2" library="freddyLibr" deviceset="USB_MICROB_PLUG_ZX64_B_5S" device=""/>
 <part name="GND" library="SparkFun-Connectors" deviceset="M01" device="PTH"/>
 <part name="3.3V" library="SparkFun-Connectors" deviceset="M01" device="PTH"/>
@@
 <part name="C2" library="SparkFun-Capacitors" deviceset="CAP" device="0805"/>
 <part name="V1" library="freddyLibr" deviceset="VOLTAGE_REGULATOR_AP2114H" device=""/>
+<part name="JP1" library="SparkFun-Connectors" deviceset="M04" device="PTH"/>
 </parts>
 <sheets>
@@
 <instances>
 <instance part="USB1" gate="G$1" x="0" y="0" rot="R90"/>
-<instance part="USB2" gate="G$1" x="0" y="-25.4" rot="MR270"/>
 <instance part="GND" gate="G$1" x="-45.72" y="12.7"/>
 <instance part="3.3V" gate="G$1" x="-55.88" y="-10.16"/>
@@
 <instance part="C2" gate="G$1" x="-17.78" y="-20.32"/>
 <instance part="V1" gate="G$1" x="-30.48" y="-10.16" rot="R90"/>
+<instance part="JP1" gate="G$1" x="2.54" y="-25.4"/>
 </instances>
 <busses>
@@
 <wire x1="10.16" y1="-5.08" x2="12.7" y2="-5.08" width="0.1524" layer="91"/>
 <wire x1="12.7" y1="-5.08" x2="12.7" y2="-12.7" width="0.1524" layer="91"/>
-<pinref part="USB2" gate="G$1" pin="VCC"/>
 <wire x1="12.7" y1="-12.7" x2="12.7" y2="-20.32" width="0.1524" layer="91"/>
-<wire x1="12.7" y1="-20.32" x2="10.16" y2="-20.32" width="0.1524" layer="91"/>
 <wire x1="-20.32" y1="-12.7" x2="-17.78" y2="-12.7" width="0.1524" layer="91"/>
 <pinref part="C2" gate="G$1" pin="1"/>
@@
 <wire x1="-17.78" y1="-12.7" x2="-17.78" y2="-15.24" width="0.1524" layer="91"/>
 <pinref part="V1" gate="G$1" pin="VIN"/>
+<pinref part="JP1" gate="G$1" pin="4"/>
+<wire x1="12.7" y1="-20.32" x2="7.62" y2="-20.32" width="0.1524" layer="91"/>
 </segment>
 </net>
@@
 <wire x1="10.16" y1="-2.54" x2="15.24" y2="-2.54" width="0.1524" layer="91"/>
 <wire x1="15.24" y1="-2.54" x2="15.24" y2="-22.86" width="0.1524" layer="91"/>
-<pinref part="USB2" gate="G$1" pin="DATA-"/>
-<wire x1="15.24" y1="-22.86" x2="10.16" y2="-22.86" width="0.1524" layer="91"/>
+<pinref part="JP1" gate="G$1" pin="3"/>
+<wire x1="15.24" y1="-22.86" x2="7.62" y2="-22.86" width="0.1524" layer="91"/>
 </segment>
 </net>
@@
 <wire x1="10.16" y1="2.54" x2="17.78" y2="2.54" width="0.1524" layer="91"/>
 <wire x1="17.78" y1="2.54" x2="17.78" y2="-25.4" width="0.1524" layer="91"/>
-<pinref part="USB2" gate="G$1" pin="DATA+"/>
-<wire x1="17.78" y1="-25.4" x2="10.16" y2="-25.4" width="0.1524" layer="91"/>
+<pinref part="JP1" gate="G$1" pin="2"/>
+<wire x1="17.78" y1="-25.4" x2="7.62" y2="-25.4" width="0.1524" layer="91"/>
 </segment>
 </net>
@@
 <pinref part="GND" gate="G$1" pin="1"/>
 <wire x1="-38.1" y1="12.7" x2="-12.7" y2="12.7" width="0.1524" layer="91"/>
-<wire x1="20.32" y1="5.08" x2="20.32" y2="-30.48" width="0.1524" layer="91"/>
-<pinref part="USB2" gate="G$1" pin="GND"/>
-<wire x1="20.32" y1="-30.48" x2="10.16" y2="-30.48" width="0.1524" layer="91"/>
+<wire x1="20.32" y1="5.08" x2="20.32" y2="-27.94" width="0.1524" layer="91"/>
+<wire x1="20.32" y1="-27.94" x2="20.32" y2="-38.1" width="0.1524" layer="91"/>
 <wire x1="-30.48" y1="-38.1" x2="20.32" y2="-38.1" width="0.1524" layer="91"/>
-<wire x1="20.32" y1="-38.1" x2="20.32" y2="-30.48" width="0.1524" layer="91"/>
 <pinref part="V1" gate="G$1" pin="GND"/>
+<pinref part="JP1" gate="G$1" pin="1"/>
+<wire x1="7.62" y1="-27.94" x2="20.32" y2="-27.94" width="0.1524" layer="91"/>
 </segment>
 </net>
